Commit message: Moved drone_controller into the Git workspace

File: 41068_ignition_bringup/urdf_drone/parrot.urdf.xacro (robot description, xacro)
@@ -16,10 +16,11 @@
                izz="3.328e-3" />
     </inertial>
-<!--     <collision name="collision">
-      <origin xyz="-0.00424 0.00014 -0.00595" rpy="0 0 0"/>
+    <!-- Add collision geometry to prevent lidar self-collision -->
+    <collision name="collision">
+      <origin xyz="0 0 0" rpy="0 0 0"/>
       <geometry>
-        <box size="0.5 0.5 0.2"/>
+        <cylinder length="0.05" radius="0.15"/>  <!-- Encompasses propellers -->
       </geometry>
-    </collision> -->
+    </collision>
     <visual name="hull">
       <geometry>
@@ -58,8 +59,28 @@
   </joint>
   <link name="imu_link"/>
+  <!-- ADD NEW LIDAR MOUNT HERE -->
+  <joint name="lidar_mount_joint" type="fixed">
+    <parent link="base_link"/>
+    <child link="lidar_mount"/>
+    <origin xyz="0 0 0.25" rpy="0 0 0"/>  <!-- Mount higher up -->
+  </joint>
+  <link name="lidar_mount">
+    <visual>
+      <geometry>
+        <cylinder length="0.03" radius="0.01"/>  <!-- Thin mounting post -->
+      </geometry>
+      <material name="dark"/>
+    </visual>
+    <inertial>
+      <mass value="0.01"/>
+      <origin xyz="0 0 0"/>
+      <inertia ixx="0.0001" iyy="0.0001" izz="0.0001" ixy="0" ixz="0" iyz="0"/>
+    </inertial>
+  </link>
+  <!-- MODIFY THE SCAN JOINT TO USE THE NEW MOUNT -->
   <joint name="scan_joint" type="fixed">
-    <parent link="base_link"/>
+    <parent link="lidar_mount"/>  <!-- Changed from base_link to lidar_mount -->
     <child link="base_scan"/>
-    <origin xyz="0 0 0.2" rpy="0 0 0"/>
+    <origin xyz="0 0 0.02" rpy="0 0 0"/>  <!-- Small offset from mount -->
   </joint>
   <link name="base_scan">
@@ -72,5 +93,5 @@
     </visual>
     <inertial>
-      <mass value="0" />
+      <mass value="0.01" />  <!-- Give it small mass -->
       <origin xyz="0 0 0" />
       <inertia ixx="0.001" ixy="0.0" ixz="0.0"
@@ -80,5 +101,5 @@
   </link>
   <joint name="camera_joint" type="fixed">
-    <origin xyz="0.25 0.0 0.25" rpy="0 0.785398 0"/> <!-- 0.5 0.0 0.9 -->
+    <origin xyz="0.25 0.0 0.25" rpy="0 0.785398 0"/>
     <parent link="base_link"/>
     <child link="camera_link"/>

Commit message: LIDAR working on drone

File: 41068_ignition_bringup/urdf_drone/parrot.urdf.xacro (robot description, xacro)
@@ -16,11 +16,10 @@
                izz="3.328e-3" />
     </inertial>
-    <!-- Add collision geometry to prevent lidar self-collision -->
-    <collision name="collision">
-      <origin xyz="0 0 0" rpy="0 0 0"/>
+<!--     <collision name="collision">
+      <origin xyz="-0.00424 0.00014 -0.00595" rpy="0 0 0"/>
       <geometry>
-        <cylinder length="0.05" radius="0.15"/>  <!-- Encompasses propellers -->
+        <box size="0.5 0.5 0.2"/>
       </geometry>
-    </collision>
+    </collision> -->
     <visual name="hull">
       <geometry>
@@ -59,28 +58,8 @@
   </joint>
   <link name="imu_link"/>
-  <!-- ADD NEW LIDAR MOUNT HERE -->
-  <joint name="lidar_mount_joint" type="fixed">
+  <joint name="scan_joint" type="fixed">
     <parent link="base_link"/>
-    <child link="lidar_mount"/>
-    <origin xyz="0 0 0.25" rpy="0 0 0"/>  <!-- Mount higher up -->
-  </joint>
-  <link name="lidar_mount">
-    <visual>
-      <geometry>
-        <cylinder length="0.03" radius="0.01"/>  <!-- Thin mounting post -->
-      </geometry>
-      <material name="dark"/>
-    </visual>
-    <inertial>
-      <mass value="0.01"/>
-      <origin xyz="0 0 0"/>
-      <inertia ixx="0.0001" iyy="0.0001" izz="0.0001" ixy="0" ixz="0" iyz="0"/>
-    </inertial>
-  </link>
-  <!-- MODIFY THE SCAN JOINT TO USE THE NEW MOUNT -->
-  <joint name="scan_joint" type="fixed">
-    <parent link="lidar_mount"/>  <!-- Changed from base_link to lidar_mount -->
     <child link="base_scan"/>
-    <origin xyz="0 0 0.02" rpy="0 0 0"/>  <!-- Small offset from mount -->
+    <origin xyz="0 0 0.2" rpy="0 0 0"/>
   </joint>
   <link name="base_scan">
@@ -93,5 +72,5 @@
     </visual>
     <inertial>
-      <mass value="0.01" />  <!-- Give it small mass -->
+      <mass value="0" />
       <origin xyz="0 0 0" />
       <inertia ixx="0.001" ixy="0.0" ixz="0.0"
@@ -101,5 +80,5 @@
   </link>
   <joint name="camera_joint" type="fixed">
-    <origin xyz="0.25 0.0 0.25" rpy="0 0.785398 0"/>
+    <origin xyz="0.25 0.0 0.25" rpy="0 0.785398 0"/> <!-- 0.5 0.0 0.9 -->
     <parent link="base_link"/>
     <child link="camera_link"/>

Commit message: Nav2 flight straighter, trees scaled up in new worldwith SLAM map, need to add LIDAR to UI

File: 41068_ignition_bringup/urdf_drone/parrot.urdf.xacro (robot description, xacro)
@@ -16,5 +16,5 @@
                izz="3.328e-3" />
     </inertial>
-<!--     <collision name="collision">
+    <!-- <collision name="collision">
       <origin xyz="-0.00424 0.00014 -0.00595" rpy="0 0 0"/>
       <geometry>

Commit message: Nav2 flight straighter, and Altitude control smoother, collisions on, Gravity on for Plantation2

File: 41068_ignition_bringup/urdf_drone/parrot.urdf.xacro (robot description, xacro)
@@ -16,10 +16,10 @@
                izz="3.328e-3" />
     </inertial>
-    <!-- <collision name="collision">
+    <collision name="collision">
       <origin xyz="-0.00424 0.00014 -0.00595" rpy="0 0 0"/>
       <geometry>
         <box size="0.5 0.5 0.2"/>
       </geometry>
-    </collision> -->
+    </collision>
     <visual name="hull">
       <geometry>
